Commit message: Add xl430 arm description and meshes

File: src/arm_description/urdf/arm.urdf.xacro (robot description, xacro)
@@ -22,18 +22,16 @@
     <visual>
       <geometry>
-        <box size="0.1 0.1 0.05"/>
-      </geometry>
-      <material name="gray"/>
-    </visual>
-    <collision>
-      <geometry>
-        <box size="0.1 0.1 0.05"/>
+        <mesh filename="package://arm_description/meshes/visual/link_0.dae"/>
+      </geometry>
+    </visual>
+    <collision>
+      <geometry>
+        <mesh filename="package://arm_description/meshes/collision/link_0.stl"/>
       </geometry>
     </collision>
     <inertial>
       <mass value="1.0"/>
-      <inertia ixx="0.01" ixy="0" ixz="0"
-               iyy="0.01" iyz="0"
-               izz="0.01"/>
+      <inertia ixx="0.01" iyy="0.01" izz="0.01"
+               ixy="0" ixz="0" iyz="0"/>
     </inertial>
   </link>
@@ -43,22 +41,20 @@
   <link name="link_1">
     <visual>
-      <geometry>
-        <cylinder length="0.15" radius="0.02"/>
-      </geometry>
-      <origin xyz="0 0 0.075"/>
-      <material name="gray"/>
-    </visual>
-    <collision>
-      <geometry>
-        <cylinder length="0.15" radius="0.02"/>
-      </geometry>
-      <origin xyz="0 0 0.075"/>
-    </collision>
-    <inertial>
-      <origin xyz="0 0 0.075"/>
+      <origin xyz="0 0 0" rpy="0 0 0"/>
+      <geometry>
+        <mesh filename="package://arm_description/meshes/visual/link_1.dae"/>
+      </geometry>
+    </visual>
+    <collision>
+      <origin xyz="0 0 0" rpy="0 0 0"/>
+      <geometry>
+        <mesh filename="package://arm_description/meshes/collision/link_1.stl"/>
+      </geometry>
+    </collision>
+    <inertial>
+      <origin xyz="0 0 0"/>
       <mass value="0.3"/>
-      <inertia ixx="0.001" ixy="0" ixz="0"
-               iyy="0.001" iyz="0"
-               izz="0.001"/>
+      <inertia ixx="0.001" iyy="0.001" izz="0.001"
+              ixy="0" ixz="0" iyz="0"/>
     </inertial>
   </link>
@@ -66,7 +62,7 @@
     <parent link="base_link"/>
     <child link="link_1"/>
-    <origin xyz="0 0 0.05"/>
-    <axis xyz="0 0 1"/>
-    <limit lower="-3.14159" upper="3.14159" effort="2.0" velocity="2.0"/>
+    <origin xyz="0 0 0.0615" rpy="0 0 0"/>
+    <axis xyz="0 0 1"/>
+    <limit lower="${-pi}" upper="${pi}" effort="2.0" velocity="2.5"/>
   </joint>
   <!-- ========================= -->
@@ -75,22 +71,20 @@
   <link name="link_2">
     <visual>
-      <geometry>
-        <cylinder length="0.15" radius="0.02"/>
-      </geometry>
-      <origin xyz="0 0 0.075"/>
-      <material name="gray"/>
-    </visual>
-    <collision>
-      <geometry>
-        <cylinder length="0.15" radius="0.02"/>
-      </geometry>
-      <origin xyz="0 0 0.075"/>
-    </collision>
-    <inertial>
-      <origin xyz="0 0 0.075"/>
+      <origin xyz="0 0 0" rpy="0 0 0"/>
+      <geometry>
+        <mesh filename="package://arm_description/meshes/visual/link_2.dae"/>
+      </geometry>
+    </visual>
+    <collision>
+      <origin xyz="0 0 0" rpy="0 0 0"/>
+      <geometry>
+        <mesh filename="package://arm_description/meshes/collision/link_2.stl"/>
+      </geometry>
+    </collision>
+    <inertial>
+      <origin xyz="0 0 0"/>
       <mass value="0.25"/>
-      <inertia ixx="0.001" ixy="0" ixz="0"
-               iyy="0.001" iyz="0"
-               izz="0.001"/>
+      <inertia ixx="0.001" iyy="0.001" izz="0.001"
+               ixy="0" ixz="0" iyz="0"/>
     </inertial>
   </link>
@@ -98,7 +92,7 @@
     <parent link="link_1"/>
     <child link="link_2"/>
-    <origin xyz="0 0 0.15"/>
-    <axis xyz="0 1 0"/>
-    <limit lower="-3.14159" upper="3.14159" effort="2.0" velocity="2.0"/>
+    <origin xyz="-0.10 0 0.18" rpy="${-pi/2} ${-pi/3} ${pi/2}"/>
+    <axis xyz="0 0 1"/>
+    <limit lower="${-pi}" upper="${pi}" effort="2.0" velocity="2.5"/>
   </joint>
   <!-- ========================= -->
@@ -107,22 +101,20 @@
   <link name="link_3">
     <visual>
-      <geometry>
-        <cylinder length="0.12" radius="0.02"/>
-      </geometry>
-      <origin xyz="0 0 0.06"/>
-      <material name="gray"/>
-    </visual>
-    <collision>
-      <geometry>
-        <cylinder length="0.12" radius="0.02"/>
-      </geometry>
-      <origin xyz="0 0 0.06"/>
-    </collision>
-    <inertial>
-      <origin xyz="0 0 0.06"/>
+      <origin xyz="0 0 0" rpy="0 0 0"/>
+      <geometry>
+        <mesh filename="package://arm_description/meshes/visual/link_3.dae"/>
+      </geometry>
+    </visual>
+    <collision>
+      <origin xyz="0 0 0" rpy="0 0 0"/>
+      <geometry>
+        <mesh filename="package://arm_description/meshes/collision/link_3.stl"/>
+      </geometry>
+    </collision>
+    <inertial>
+      <origin xyz="0 0 0.075"/>
       <mass value="0.2"/>
-      <inertia ixx="0.0008" ixy="0" ixz="0"
-               iyy="0.0008" iyz="0"
-               izz="0.0008"/>
+      <inertia ixx="0.0008" iyy="0.0008" izz="0.0008"
+               ixy="0" ixz="0" iyz="0"/>
     </inertial>
   </link>
@@ -130,85 +122,186 @@
     <parent link="link_2"/>
     <child link="link_3"/>
-    <origin xyz="0 0 0.15"/>
-    <axis xyz="0 1 0"/>
-    <limit lower="-3.14159" upper="3.14159" effort="2.0" velocity="2.0"/>
+    <origin xyz="0.69 0 0.04" rpy="0 ${pi} ${3*pi/2}"/>
+    <axis xyz="0 0 1"/>
+    <limit lower="${-pi}" upper="${pi}" effort="2.0" velocity="2.5"/>
+  </joint>
+  <!-- ========================= -->
+  <!--        LINK 4             -->
+  <!-- ========================= -->
+  <link name="link_4">
+    <visual>
+      <origin xyz="0 0 0" rpy="0 0 0"/>
+      <geometry>
+        <mesh filename="package://arm_description/meshes/visual/link_4.dae"/>
+      </geometry>
+    </visual>
+    <collision>
+      <origin xyz="0 0 0" rpy="0 0 0"/>
+      <geometry>
+        <mesh filename="package://arm_description/meshes/collision/link_4.stl"/>
+      </geometry>
+    </collision>
+    <inertial>
+      <origin xyz="0 0 0.05"/>
+      <mass value="0.15"/>
+      <inertia ixx="0.0004" iyy="0.0004" izz="0.0004"
+               ixy="0" ixz="0" iyz="0"/>
+    </inertial>
+  </link>
+  <joint name="joint_4" type="revolute">
+    <parent link="link_3"/>
+    <child link="link_4"/>
+    <origin xyz="0.52 0 0.07" rpy="0 ${pi} ${pi + pi/6}"/>
+    <axis xyz="0 0 1"/>
+    <limit lower="${-pi}" upper="${pi}" effort="1.5" velocity="2.0"/>
+  </joint>
+  <!-- ========================= -->
+  <!--        LINK 5             -->
+  <!-- ========================= -->
+  <link name="link_5">
+    <visual>
+      <origin xyz="0 0 0" rpy="0 0 0"/>
+      <geometry>
+        <mesh filename="package://arm_description/meshes/visual/link_5.dae"/>
+      </geometry>
+    </visual>
+    <collision>
+      <origin xyz="0 0 0" rpy="0 0 0"/>
+      <geometry>
+        <mesh filename="package://arm_description/meshes/collision/link_5.stl"/>
+      </geometry>
+    </collision>
+    <inertial>
+      <origin xyz="0 0 0.04"/>
+      <mass value="0.12"/>
+      <inertia ixx="0.0003" iyy="0.0003" izz="0.0003"
+               ixy="0" ixz="0" iyz="0"/>
+    </inertial>
+  </link>
+  <joint name="joint_5" type="revolute">
+    <parent link="link_4"/>
+    <child link="link_5"/>
+    <origin xyz="0.11 0 0.11" rpy="${pi/2} ${pi} ${pi/2}"/>
+    <axis xyz="0 0 1"/>
+    <limit lower="${-5*pi/6}" upper="${5*pi/6}" effort="1.2" velocity="2.0"/>
+  </joint>
+  <!-- ========================= -->
+  <!--        LINK 6             -->
+  <!-- ========================= -->
+  <link name="link_6">
+    <visual>
+      <origin xyz="0 0 0" rpy="0 0 0"/>
+      <geometry>
+        <mesh filename="package://arm_description/meshes/visual/link_6.dae"/>
+      </geometry>
+    </visual>
+    <collision>
+      <origin xyz="0 0 0" rpy="0 0 0"/>
+      <geometry>
+        <mesh filename="package://arm_description/meshes/collision/link_6.stl"/>
+      </geometry>
+    </collision>
+    <inertial>
+      <mass value="0.05"/>
+      <inertia ixx="0.0001" iyy="0.0001" izz="0.0001"
+               ixy="0" ixz="0" iyz="0"/>
+    </inertial>
+  </link>
+  <joint name="joint_6" type="revolute">
+    <parent link="link_5"/>
+    <child link="link_6"/>
+    <origin xyz="-0.086 0 0.133" rpy="0 ${-pi/2} 0"/>
+    <axis xyz="0 0 1"/>
+    <limit lower="${-pi}" upper="${pi}" effort="1.0" velocity="2.5"/>
   </joint>
   <!-- ================================================= -->
   <!--                ROS 2 CONTROL                     -->
   <!-- ================================================= -->
-  <ros2_control name="DynamixelSystem" type="system">
-    <hardware>
-      <plugin>dynamixel_hardware_interface/DynamixelHardware</plugin>
-      <param name="port_name">/dev/ttyACM0</param>
-      <param name="baud_rate">1000000</param>
-      <param name="number_of_joints">3</param>
-      <param name="number_of_transmissions">3</param>
-      <param name="disable_torque_at_init">true</param>
-      <!-- Path relative to package share -->
-      <param name="dynamixel_model_folder">/param/dxl_model</param>
-    </hardware>
-    <!-- Joint interfaces -->
-    <joint name="joint_1">
-      <command_interface name="position"/>
-      <state_interface name="position"/>
-      <state_interface name="velocity"/>
-    </joint>
-    <joint name="joint_2">
-      <command_interface name="position"/>
-      <state_interface name="position"/>
-      <state_interface name="velocity"/>
-    </joint>
-    <joint name="joint_3">
-      <command_interface name="position"/>
-      <state_interface name="position"/>
-      <state_interface name="velocity"/>
-    </joint>
-    <!-- Transmissions -->
-    <transmission name="trans_1">
-      <plugin>transmission_interface/SimpleTransmission</plugin>
-      <joint name="joint_1" role="joint"/>
-      <actuator name="dxl1" role="actuator">
-        <command_interface name="position"/>
-        <mechanical_reduction>1</mechanical_reduction>
-      </actuator>
-    </transmission>
-    <transmission name="trans_2">
-      <plugin>transmission_interface/SimpleTransmission</plugin>
-      <joint name="joint_2" role="joint"/>
-      <actuator name="dxl2" role="actuator">
-        <command_interface name="position"/>
-        <mechanical_reduction>1</mechanical_reduction>
-      </actuator>
-    </transmission>
-    <transmission name="trans_3">
-      <plugin>transmission_interface/SimpleTransmission</plugin>
-      <joint name="joint_3" role="joint"/>
-      <actuator name="dxl3" role="actuator">
-        <command_interface name="position"/>
-        <mechanical_reduction>1</mechanical_reduction>
-      </actuator>
-    </transmission>
-    <!-- Dynamixels -->
-    <gpio name="dxl1">
-      <param name="type">dxl</param>
-      <param name="ID">1</param>
-      <command_interface name="Goal Position"/>
-      <state_interface name="Present Position"/>
-      <state_interface name="Present Velocity"/>
-    </gpio>
-    <gpio name="dxl2">
-      <param name="type">dxl</param>
-      <param name="ID">2</param>
-      <command_interface name="Goal Position"/>
-      <state_interface name="Present Position"/>
-      <state_interface name="Present Velocity"/>
-    </gpio>
-    <gpio name="dxl3">
-      <param name="type">dxl</param>
-      <param name="ID">3</param>
-      <command_interface name="Goal Position"/>
-      <state_interface name="Present Position"/>
-      <state_interface name="Present Velocity"/>
-    </gpio>
-  </ros2_control>
+<ros2_control name="DynamixelSystem" type="system">
+  <hardware>
+    <plugin>dynamixel_hardware_interface/DynamixelHardware</plugin>
+    <!-- Communication -->
+    <param name="port_name">/dev/ttyACM0</param>
+    <param name="baud_rate">1000000</param>
+    <param name="protocol_version">2.0</param>
+    <param name="error_timeout_ms">100</param>
+    <!-- Control -->
+    <param name="control_mode">position</param>
+    <!-- Robot structure -->
+    <param name="number_of_joints">6</param>
+    <param name="number_of_transmissions">6</param>
+    <param name="joint_names">joint_1 joint_2 joint_3 joint_4 joint_5 joint_6</param>
+    <param name="joint_ids">1 2 3 4 5 6</param>
+    <param name="joint_models">xl430_w250 xl430_w250 xl430_w250 xl430_w250 xl430_w250 xl430_w250</param>
+    <!-- Dynamixel model database -->
+    <param name="dynamixel_model_folder">/param/dxl_model</param>
+  </hardware>
+  <!-- Joint definitions -->
+  <joint name="joint_1">
+    <command_interface name="position"/>
+    <state_interface name="position"/>
+    <state_interface name="velocity"/>
+  </joint>
+  <joint name="joint_2">
+    <command_interface name="position"/>
+    <state_interface name="position"/>
+    <state_interface name="velocity"/>
+  </joint>
+  <joint name="joint_3">
+    <command_interface name="position"/>
+    <state_interface name="position"/>
+    <state_interface name="velocity"/>
+  </joint>
+    <joint name="joint_4">
+    <command_interface name="position"/>
+    <state_interface name="position"/>
+    <state_interface name="velocity"/>
+  </joint>
+    <joint name="joint_5">
+    <command_interface name="position"/>
+    <state_interface name="position"/>
+    <state_interface name="velocity"/>
+  </joint>
+    <joint name="joint_6">
+    <command_interface name="position"/>
+    <state_interface name="position"/>
+    <state_interface name="velocity"/>
+  </joint>
+  <gpio name="dxl_1">
+    <param name="ID">1</param>
+    <param name="type">dxl</param>
+    <command_interface name="Goal Position"/>
+    <state_interface name="Present Position"/>
+  </gpio>
+  <gpio name="dxl_2">
+    <param name="ID">2</param>
+    <param name="type">dxl</param>
+    <command_interface name="Goal Position"/>
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
File: src/arm_moveit_config/config/xl430_arm.ros2_control.xacro (robot description, xacro)
@@ -2,5 +2,5 @@
 <robot xmlns:xacro="http://www.ros.org/wiki/xacro">
     <xacro:macro name="xl430_arm_ros2_control" params="name initial_positions_file">
-        <xacro:property name="initial_positions" value="${xacro.load_yaml(initial_positions_file)['initial_positions']}"/>
+        <xacro:property name="initial_positions" value="${load_yaml(initial_positions_file)['initial_positions']}"/>
         <ros2_control name="${name}" type="system">
             <hardware>
@@ -29,4 +29,25 @@
                 <state_interface name="velocity"/>
             </joint>
+            <joint name="joint_4">
+                <command_interface name="position"/>
+                <state_interface name="position">
+                  <param name="initial_value">${initial_positions['joint_4']}</param>
+                </state_interface>
+                <state_interface name="velocity"/>
+            </joint>
+            <joint name="joint_5">
+                <command_interface name="position"/>
+                <state_interface name="position">
+                  <param name="initial_value">${initial_positions['joint_5']}</param>
+                </state_interface>
+                <state_interface name="velocity"/>
+            </joint>
+            <joint name="joint_6">
+                <command_interface name="position"/>
+                <state_interface name="position">
+                  <param name="initial_value">${initial_positions['joint_6']}</param>
+                </state_interface>
+                <state_interface name="velocity"/>
+            </joint>
         </ros2_control>
     </xacro:macro>
